Commit message: romeo_bad: Squirrel the error away at the end

File: test/romeo/romeo_bad.urdf (robot description, URDF)
Before this commit: robot romeo, 68 links, 67 joints
Links:
- removed link body asdf
- added link body, mass 4.16277; collision mesh filename=package://romeo_description/meshes/Waist.dae; visual mesh filename=package://romeo_description/meshes/Waist.dae
Joints:
- joint REyeYaw: limit lower=-0.523598766666667 upper=0.523598766666667 effort=0 velocity=0 -> lower=-0.5235___98766666667 upper=0.523598766666667 effort=0 velocity=0
